File: EE 201 Lab 4 Exercise 1/EE 201 Lab 4 Exercise 1.kicad_sch (KiCad schematic)
At the start: 6 parts, among them SW1 Switch

Commit message: Updated PCB Files
Parts:
- C1: footprint (none) -> Capacitor_THT:C_Radial_D5.0mm_H5.0mm_P2.00mm
- D1: footprint (none) -> LED_THT:LED_D5.0mm
- R1, R2: footprint (none) -> Resistor_THT:R_Axial_DIN0516_L15.5mm_D5.0mm_P20.32mm_Horizontal
- SW1: footprint (none) -> Button_Switch_THT:SW_E-Switch_EG1224_SPDT_Angled
- V1: footprint (none) -> Connector_JST:JST_PH_B2B-PH-K_1x02_P2.00mm_Vertical
Changed lines of the file:
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@@
       (effects (font (size 1.27 1.27)) (justify left))
     )
-    (property "Footprint" "" (id 2) (at 129.2352 97.79 0)
+    (property "Footprint" "Capacitor_THT:C_Radial_D5.0mm_H5.0mm_P2.00mm" (id 2) (at 129.2352 97.79 0)
       (effects (font (size 1.27 1.27)) hide)
     )
@@
       (effects (font (size 1.27 1.27)) (justify left))
     )
-    (property "Footprint" "" (id 2) (at 149.352 95.25 90)
+    (property "Footprint" "Resistor_THT:R_Axial_DIN0516_L15.5mm_D5.0mm_P20.32mm_Horizontal" (id 2) (at 149.352 95.25 90)
       (effects (font (size 1.27 1.27)) hide)
     )
@@
     (property "Reference" "R2" (id 0) (at 104.14 78.74 90))
     (property "Value" "2.2 kOhms" (id 1) (at 104.14 81.28 90))
-    (property "Footprint" "" (id 2) (at 104.14 83.312 90)
+    (property "Footprint" "Resistor_THT:R_Axial_DIN0516_L15.5mm_D5.0mm_P20.32mm_Horizontal" (id 2) (at 104.14 83.312 90)
       (effects (font (size 1.27 1.27)) hide)
     )
@@
     (property "Reference" "SW1" (id 0) (at 119.38 77.47 0))
     (property "Value" "Switch" (id 1) (at 119.38 80.01 0))
-    (property "Footprint" "" (id 2) (at 119.38 85.09 0)
+    (property "Footprint" "Button_Switch_THT:SW_E-Switch_EG1224_SPDT_Angled" (id 2) (at 119.38 85.09 0)
       (effects (font (size 1.27 1.27)) hide)
     )
@@
     (property "Reference" "V1" (id 0) (at 89.535 90.17 0))
     (property "Value" "9 V" (id 1) (at 89.535 92.71 0))
-    (property "Footprint" "" (id 2) (at 88.9 95.25 0)
+    (property "Footprint" "Connector_JST:JST_PH_B2B-PH-K_1x02_P2.00mm_Vertical" (id 2) (at 88.9 95.25 0)
       (effects (font (size 1.27 1.27)) hide)
     )
@@
       (effects (font (size 1.27 1.27)) (justify right))
     )
-    (property "Footprint" "" (id 2) (at 151.13 105.41 0)
+    (property "Footprint" "LED_THT:LED_D5.0mm" (id 2) (at 151.13 105.41 0)
       (effects (font (size 1.27 1.27)) hide)
     )
@@
   (symbol_instances
     (path "/1b782eb2-235f-4415-a4b7-da133c6a1016"
-      (reference "C1") (unit 1) (value "4.7 uF") (footprint "")
+      (reference "C1") (unit 1) (value "4.7 uF") (footprint "Capacitor_THT:C_Radial_D5.0mm_H5.0mm_P2.00mm")
     )
     (path "/df74af7a-e333-4559-8672-b3d9201671d4"
-      (reference "D1") (unit 1) (value "LED") (footprint "")
+      (reference "D1") (unit 1) (value "LED") (footprint "LED_THT:LED_D5.0mm")
     )
     (path "/3abe0e03-368d-4bc6-b217-db3e23ed8c01"
-      (reference "R1") (unit 1) (value "20 kOhms") (footprint "")
+      (reference "R1") (unit 1) (value "20 kOhms") (footprint "Resistor_THT:R_Axial_DIN0516_L15.5mm_D5.0mm_P20.32mm_Horizontal")
     )
     (path "/8494bbf0-a700-4384-aa40-7556431a99bd"
-      (reference "R2") (unit 1) (value "2.2 kOhms") (footprint "")
+      (reference "R2") (unit 1) (value "2.2 kOhms") (footprint "Resistor_THT:R_Axial_DIN0516_L15.5mm_D5.0mm_P20.32mm_Horizontal")
     )
     (path "/9a6df613-110f-47ab-ad5b-db0bd64006fd"
-      (reference "SW1") (unit 1) (value "Switch") (footprint "")
+      (reference "SW1") (unit 1) (value "Switch") (footprint "Button_Switch_THT:SW_E-Switch_EG1224_SPDT_Angled")
     )
     (path "/bfeae824-ff86-47d9-ad60-92c81b75188c"
-      (reference "V1") (unit 1) (value "9 V") (footprint "")
+      (reference "V1") (unit 1) (value "9 V") (footprint "Connector_JST:JST_PH_B2B-PH-K_1x02_P2.00mm_Vertical")
     )
   )
