File: EE 201 Lab 4 Exercise 2/EE 201 Lab 4 Exercise 2.kicad_sch (KiCad schematic)
At the start: 10 parts, among them J1 Connector, U1 Timer

Commit message: Updated PCB Files
Parts:
- C1: footprint (none) -> Capacitor_Tantalum_SMD:CP_EIA-3216-18_Kemet-A_Pad1.58x1.35mm_HandSolder
- C2: footprint (none) -> Capacitor_SMD:C_0805_2012Metric_Pad1.18x1.45mm_HandSolder
- D1, D2: footprint (none) -> LED_SMD:LED_1206_3216Metric_Pad1.42x1.75mm_HandSolder
- J1: footprint (none) -> TerminalBlock:TerminalBlock_bornier-2_P5.08mm
- R1, R2, R3, R4: footprint (none) -> Resistor_SMD:R_0805_2012Metric_Pad1.20x1.40mm_HandSolder
- U1: footprint Package_SO:SOIC-8_3.9x4.9mm_P1.27mm -> Package_SO:SOIC-8-1EP_3.9x4.9mm_P1.27mm_EP2.29x3mm
Changed lines of the file:
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@@
       (effects (font (size 1.27 1.27)) (justify right))
     )
-    (property "Footprint" "" (id 2) (at 140.97 77.47 0)
+    (property "Footprint" "TerminalBlock:TerminalBlock_bornier-2_P5.08mm" (id 2) (at 140.97 77.47 0)
       (effects (font (size 1.27 1.27)) hide)
     )
@@
       (effects (font (size 1.27 1.27)) (justify right))
     )
-    (property "Footprint" "" (id 2) (at 96.52 135.89 0)
+    (property "Footprint" "LED_SMD:LED_1206_3216Metric_Pad1.42x1.75mm_HandSolder" (id 2) (at 96.52 135.89 0)
       (effects (font (size 1.27 1.27)) hide)
     )
@@
       (effects (font (size 1.27 1.27)) (justify left))
     )
-    (property "Footprint" "" (id 2) (at 126.6952 125.73 0)
+    (property "Footprint" "Capacitor_SMD:C_0805_2012Metric_Pad1.18x1.45mm_HandSolder" (id 2) (at 126.6952 125.73 0)
       (effects (font (size 1.27 1.27)) hide)
     )
@@
       (effects (font (size 1.27 1.27)) (justify left))
     )
-    (property "Footprint" "" (id 2) (at 94.742 102.87 90)
+    (property "Footprint" "Resistor_SMD:R_0805_2012Metric_Pad1.20x1.40mm_HandSolder" (id 2) (at 94.742 102.87 90)
       (effects (font (size 1.27 1.27)) hide)
     )
@@
   (symbol (lib_id "power:+9V") (at 143.51 86.36 0) (unit 1)
     (in_bom yes) (on_board yes) (fields_autoplaced)
-    (property "Reference" "#PWR?" (id 0) (at 143.51 90.17 0)
+    (property "Reference" "#PWR0101" (id 0) (at 143.51 90.17 0)
       (effects (font (size 1.27 1.27)) hide)
     )
@@
       (effects (font (size 1.27 1.27)) (justify left))
     )
-    (property "Footprint" "" (id 2) (at 179.832 99.06 90)
+    (property "Footprint" "Resistor_SMD:R_0805_2012Metric_Pad1.20x1.40mm_HandSolder" (id 2) (at 179.832 99.06 90)
       (effects (font (size 1.27 1.27)) hide)
     )
@@
   (symbol (lib_id "power:+9V") (at 96.52 81.28 0) (unit 1)
     (in_bom yes) (on_board yes) (fields_autoplaced)
-    (property "Reference" "#PWR?" (id 0) (at 96.52 85.09 0)
+    (property "Reference" "#PWR0106" (id 0) (at 96.52 85.09 0)
       (effects (font (size 1.27 1.27)) hide)
     )
@@
       (effects (font (size 1.27 1.27)) (justify left))
     )
-    (property "Footprint" "Package_SO:SOIC-8_3.9x4.9mm_P1.27mm" (id 2) (at 165.1 113.03 0)
+    (property "Footprint" "Package_SO:SOIC-8-1EP_3.9x4.9mm_P1.27mm_EP2.29x3mm" (id 2) (at 165.1 113.03 0)
       (effects (font (size 1.27 1.27)) hide)
     )
@@
   (symbol (lib_id "power:GND") (at 143.51 67.31 180) (unit 1)
     (in_bom yes) (on_board yes)
-    (property "Reference" "#PWR?" (id 0) (at 143.51 60.96 0)
+    (property "Reference" "#PWR0103" (id 0) (at 143.51 60.96 0)
       (effects (font (size 1.27 1.27)) hide)
     )
@@
       (effects (font (size 1.27 1.27)) (justify left))
     )
-    (property "Footprint" "" (id 2) (at 94.742 118.11 90)
+    (property "Footprint" "Resistor_SMD:R_0805_2012Metric_Pad1.20x1.40mm_HandSolder" (id 2) (at 94.742 118.11 90)
       (effects (font (size 1.27 1.27)) hide)
     )
@@
       (effects (font (size 1.27 1.27)) (justify left))
     )
-    (property "Footprint" "" (id 2) (at 182.5752 132.08 0)
+    (property "Footprint" "Capacitor_Tantalum_SMD:CP_EIA-3216-18_Kemet-A_Pad1.58x1.35mm_HandSolder" (id 2) (at 182.5752 132.08 0)
       (effects (font (size 1.27 1.27)) hide)
     )
@@
   (symbol (lib_id "power:+9V") (at 140.97 67.31 0) (unit 1)
     (in_bom yes) (on_board yes) (fields_autoplaced)
-    (property "Reference" "#PWR?" (id 0) (at 140.97 71.12 0)
+    (property "Reference" "#PWR0102" (id 0) (at 140.97 71.12 0)
       (effects (font (size 1.27 1.27)) hide)
     )
@@
       (effects (font (size 1.27 1.27)) (justify left))
     )
-    (property "Footprint" "" (id 2) (at 179.832 87.63 90)
+    (property "Footprint" "Resistor_SMD:R_0805_2012Metric_Pad1.20x1.40mm_HandSolder" (id 2) (at 179.832 87.63 90)
       (effects (font (size 1.27 1.27)) hide)
     )
@@
   (symbol (lib_id "power:+9V") (at 181.61 83.82 0) (unit 1)
     (in_bom yes) (on_board yes) (fields_autoplaced)
-    (property "Reference" "#PWR?" (id 0) (at 181.61 87.63 0)
+    (property "Reference" "#PWR0104" (id 0) (at 181.61 87.63 0)
       (effects (font (size 1.27 1.27)) hide)
     )
@@
       (effects (font (size 1.27 1.27)) (justify right))
     )
-    (property "Footprint" "" (id 2) (at 96.52 85.09 0)
+    (property "Footprint" "LED_SMD:LED_1206_3216Metric_Pad1.42x1.75mm_HandSolder" (id 2) (at 96.52 85.09 0)
       (effects (font (size 1.27 1.27)) hide)
     )
@@
   (symbol (lib_id "power:GND") (at 137.16 147.32 0) (unit 1)
     (in_bom yes) (on_board yes) (fields_autoplaced)
-    (property "Reference" "#PWR?" (id 0) (at 137.16 153.67 0)
+    (property "Reference" "#PWR0105" (id 0) (at 137.16 153.67 0)
       (effects (font (size 1.27 1.27)) hide)
     )
@@
   (symbol_instances
     (path "/45507001-a609-43aa-8c58-8d7079fe37d9"
-      (reference "#PWR?") (unit 1) (value "+9V") (footprint "")
+      (reference "#PWR0101") (unit 1) (value "+9V") (footprint "")
+    )
+    (path "/c98c876b-b092-451f-b1cf-cd6b501af8b3"
+      (reference "#PWR0102") (unit 1) (value "+9V") (footprint "")
+    )
+    (path "/614944db-a36f-4086-b311-8c18778185d2"
+      (reference "#PWR0103") (unit 1) (value "GND") (footprint "")
+    )
+    (path "/dc9b52e7-c02b-48d4-877d-51e3bda9c399"
+      (reference "#PWR0104") (unit 1) (value "+9V") (footprint "")
+    )
+    (path "/eba5f0b2-1834-46fa-9dc2-366e496e8e43"
+      (reference "#PWR0105") (unit 1) (value "GND") (footprint "")
     )
     (path "/58706176-e371-44a9-bac4-2efb0d684948"
-      (reference "#PWR?") (unit 1) (value "+9V") (footprint "")
-    )
-    (path "/614944db-a36f-4086-b311-8c18778185d2"
-      (reference "#PWR?") (unit 1) (value "GND") (footprint "")
-    )
-    (path "/c98c876b-b092-451f-b1cf-cd6b501af8b3"
-      (reference "#PWR?") (unit 1) (value "+9V") (footprint "")
-    )
-    (path "/dc9b52e7-c02b-48d4-877d-51e3bda9c399"
-      (reference "#PWR?") (unit 1) (value "+9V") (footprint "")
-    )
-    (path "/eba5f0b2-1834-46fa-9dc2-366e496e8e43"
-      (reference "#PWR?") (unit 1) (value "GND") (footprint "")
+      (reference "#PWR0106") (unit 1) (value "+9V") (footprint "")
     )
     (path "/bbc4cf20-1eb9-4111-a923-293d89252318"
-      (reference "C1") (unit 1) (value "10 uF") (footprint "")
+      (reference "C1") (unit 1) (value "10 uF") (footprint "Capacitor_Tantalum_SMD:CP_EIA-3216-18_Kemet-A_Pad1.58x1.35mm_HandSolder")
     )
     (path "/3ec3f434-16be-41c0-9af5-09607b1c38a0"
-      (reference "C2") (unit 1) (value "0.01 uF") (footprint "")
+      (reference "C2") (unit 1) (value "0.01 uF") (footprint "Capacitor_SMD:C_0805_2012Metric_Pad1.18x1.45mm_HandSolder")
     )
     (path "/e2c06c30-a416-4194-8346-d318f9f84d9b"
-      (reference "D1") (unit 1) (value "LED") (footprint "")
+      (reference "D1") (unit 1) (value "LED") (footprint "LED_SMD:LED_1206_3216Metric_Pad1.42x1.75mm_HandSolder")
     )
     (path "/2dc6e577-f966-4483-b156-697886ada2fc"
-      (reference "D2") (unit 1) (value "LED") (footprint "")
+      (reference "D2") (unit 1) (value "LED") (footprint "LED_SMD:LED_1206_3216Metric_Pad1.42x1.75mm_HandSolder")
     )
     (path "/1b336aed-4c02-4614-993e-30df816cacf2"
-      (reference "J1") (unit 1) (value "Connector") (footprint "")
+      (reference "J1") (unit 1) (value "Connector") (footprint "TerminalBlock:TerminalBlock_bornier-2_P5.08mm")
     )
     (path "/d8f0cf10-c91c-40df-80e2-025b1663e153"
-      (reference "R1") (unit 1) (value "1 kOhms") (footprint "")
+      (reference "R1") (unit 1) (value "1 kOhms") (footprint "Resistor_SMD:R_0805_2012Metric_Pad1.20x1.40mm_HandSolder")
     )
     (path "/4ef72730-13a3-41e0-8826-2a19531ca1bf"
-      (reference "R2") (unit 1) (value "10 kOhms") (footprint "")
+      (reference "R2") (unit 1) (value "10 kOhms") (footprint "Resistor_SMD:R_0805_2012Metric_Pad1.20x1.40mm_HandSolder")
     )
     (path "/43c8b0f9-9574-445a-932a-4b62f55a8dda"
-      (reference "R3") (unit 1) (value "1 kOhms") (footprint "")
+      (reference "R3") (unit 1) (value "1 kOhms") (footprint "Resistor_SMD:R_0805_2012Metric_Pad1.20x1.40mm_HandSolder")
     )
     (path "/9047a31c-7641-4a4e-8fc4-678087127545"
-      (reference "R4") (unit 1) (value "1 kOhms") (footprint "")
+      (reference "R4") (unit 1) (value "1 kOhms") (footprint "Resistor_SMD:R_0805_2012Metric_Pad1.20x1.40mm_HandSolder")
     )
     (path "/593f3ea8-f54f-4ba5-a92b-4bf27f1e53d0"
-      (reference "U1") (unit 1) (value "Timer") (footprint "Package_SO:SOIC-8_3.9x4.9mm_P1.27mm")
-    )
-  )
+      (reference "U1") (unit 1) (value "Timer") (footprint "Package_SO:SOIC-8-1EP_3.9x4.9mm_P1.27mm_EP2.29x3mm")
+    )
+  )
